File: Alchitry_Element_Template/Alchitry_Element_Template.kicad_pcb (KiCad board)
At the start: 2 copper layers, 65 x 45 mm, 1 part

Commit message: add pin names to au symbol
Parts:
- B1: value ALCHITRY_ELEMENT_AU -> Alchitry_Element_AU; footprint ALCHITRY_ELEMENT:ELEMENT -> Alchitry_Element:Element
